File: Matrix_Rev3-2.sch (KiCad schematic (older format))
At the start: 34 parts, among them SW1 DPST, SW10 DPST, SW11 DPST, SW12 DPST, SW13 DPST, SW14 DPST, SW15 DPST, SW16 DPST, SW2 DPST, SW3 DPST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

Commit message: Started track tracing
Connections:
- net c1: now also D13.2 (K), D5.2 (K), D9.2 (K); no longer D2.2 (K), D3.2 (K), D4.2 (K)
- net c2: now also D10.2 (K), D14.2 (K), D2.2 (K); no longer D5.2 (K), D7.2 (K), D8.2 (K)
- net c3: now also D15.2 (K), D3.2 (K), D7.2 (K); no longer D10.2 (K), D12.2 (K), D9.2 (K)
- net c4: now also D12.2 (K), D4.2 (K), D8.2 (K); no longer D13.2 (K), D14.2 (K), D15.2 (K)
Changed lines of the file:
@@
-EESchema Schematic File Version 2  date Onsdag 21 Augusti 2013 18:57:07
+EESchema Schematic File Version 2  date Onsdag 21 Augusti 2013 19:38:09
 LIBS:power
 LIBS:device
@@
 	2750 2800 3100 2800
 Text Label 2650 2700 0    60   ~ 0
-c1
+c2
 Text Label 3350 2700 0    60   ~ 0
-c1
+c3
 Text Label 3950 2700 0    60   ~ 0
-c1
+c4
 Text Label 1900 1100 0    60   ~ 0
 a1
@@
 a2
 Text Label 4550 2700 0    60   ~ 0
-c2
+c1
 Text Label 9050 1550 0    60   ~ 0
 a[1..4]
@@
 c2
 Text Label 6000 2700 0    60   ~ 0
-c2
+c3
 Text Label 6750 2700 0    60   ~ 0
-c2
+c4
 Text Label 5250 1100 0    60   ~ 0
 a2
@@
 	2000 4750 2000 4700
 Text Label 2750 4750 0    60   ~ 0
-c3
+c2
 Text Label 3450 4750 0    60   ~ 0
 c3
 Text Label 4050 4750 0    60   ~ 0
-c3
+c4
 Text Label 2000 3150 0    60   ~ 0
 a3
@@
 a3
 Text Label 2000 4750 0    60   ~ 0
-c3
+c1
 Wire Wire Line
 	3450 4700 3450 4750
@@
 a4
 Text Label 4650 4750 0    60   ~ 0
-c4
+c1
 Text Label 7050 4850 0    60   ~ 0
 c[3..4]
@@
 	6750 3000 6850 3100
 Text Label 5350 4750 0    60   ~ 0
-c4
+c2
 Text Label 6100 4750 0    60   ~ 0
-c4
+c3
 Text Label 6850 4750 0    60   ~ 0
 c4
