File: LAYOUT_A4.sch (KiCad schematic (older format))
At the start: 108 parts, among them SW1 DPST, SW10 DPST, SW11 DPST, SW12 DPST, SW13 DPST, SW14 DPST, SW15 DPST, SW16 DPST, SW2 DPST, SW3 DPST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

Commit message: MIDI I/O added
Parts:
- added D?: DIODE, ~, symbol DIODE
- added MIDIIN1, MIDIOUT1: DIN_5, symbol DIN_5
- added R? (x2): 220, ~, symbol R
- added R?: 3.3k, ~, symbol R
- added R?: 100k, ~, symbol R
- added U?: OPTO-TRANSISTOR, symbol OPTO-TRANSISTOR
Connections:
- net GND: now also MIDIOUT1.3, R?.1, U?.4 (E)
- new net: MIDIOUT1.4, R?.2
- new net: D?.1 (A), MIDIIN1.2, U?.2 (K)
- new net: MIDIIN1.4, R?.2
- new net: R?.2, U?.6 (B)
- new net: D?.2 (K), R?.1, U?.1 (A)
- new net MIDIIN: R?.2, U?.5 (C)
- new net MIDIOUT: MIDIOUT1.2
- new net VCC: R?.1, R?.1
- no-connect marks 0 -> 5
Other:
- moved on the sheet: COLS1, ROWS1

Commit message: MIDI ports added
Parts:
- removed R?: 100k, ~, symbol R
- added IOIO1: ATMEGA88-A, TQFP32, symbol ATMEGA88-A
- added K1: CONN_3, symbol CONN_3
- added MIDITHRU1: DIN_5, symbol DIN_5
- added R19, R23, R24: 220, ~, symbol R
- added U1: 4049, symbol 4049
- R22: renamed from R?; value 3.3k -> 280
- gave numbers to parts that had none: 4
Connections:
- net GND: now also MIDITHRU1.3, U1.8 (VSS), U1.8 (VSS), U1.8 (VSS), U1.8 (VSS)
- net MIDIIN: now also K1.1 (P1), U1.7
- net MIDIOUT: now also K1.2 (PM), U1.5; no longer MIDIOUT1.2
- net VCC: now also U2.6 (B), K1.3 (P3), R24.1, U1.1 (VCC), U1.1 (VCC), U1.1 (VCC), U1.1 (VCC)
- new net: MIDIOUT1.2, R19.1
- new net: R19.2, U1.2
- new net: U1.6, U1.9
- new net: R23.1, U1.10
- new net: U1.3, U1.4
- new net: MIDITHRU1.2, R23.2
- new net: MIDITHRU1.4, R24.2
- no-connect marks 5 -> 40
Other:
- moved on the sheet: D35, MIDIIN1, MIDIOUT1, R20, R21, R22, U2
